Commit message: Fixed xacro for urdf -> sdf generation

File: trackbot_gazebo/models/trackbot_sensors/sensors.xacro (robot description, xacro)
@@ -1,4 +1,4 @@
 <?xml version="1.0"?>
-<sdf version="1.6" xmlns:xacro="http://ros.org/wiki/xacro">
+<robot xmlns:xacro="http://ros.org/wiki/xacro">
   <xacro:macro name="camera_sensor" params="sensor_name parent_link pose rpy">
     <link name="${sensor_name}_link">
@@ -6,7 +6,8 @@
       <visual name="${sensor_name}_visual">
         <geometry>
-          <box><size>0.05 0.05 0.05</size></box>
+          <box size="0.05 0.05 0.05"/>
         </geometry>
-        <material>
+        <material name="camera_color">
+          <color rgba="0.5 0.5 0.5 1.0"/>
           <ambient>1.0 1.0 0.0 1.0</ambient>
           <diffuse>1.0 1.0 0.0 1.0</diffuse>
@@ -16,9 +17,12 @@
       </visual>
       <inertial>
-        <mass>0.1</mass>
-        <inertia>
+        <mass value="0.1"/>
+        <inertia ixx="0.1" ixy="0.0" ixz="0.0"
+           iyy="0.1" iyz="0.0"
+           izz="0.1"/>
+        <!--<inertia>
           <ixx>1e-5</ixx><iyy>1e-5</iyy><izz>1e-5</izz>
           <ixy>0</ixy><ixz>0</ixz><iyz>0</iyz>
-        </inertia>
+        </inertia>-->
       </inertial>
       <sensor name="${sensor_name}" type="camera">
@@ -37,10 +41,8 @@
     </link>
     <joint name="${sensor_name}_joint" type="fixed">
-      <parent>${parent_link}</parent>
-      <child>${sensor_name}_link</child>
-      <pose>0 0 0 0 0 0</pose>
-      <axis>
-        <xyz>0 0 1</xyz>
-      </axis>
+      <origin xyz="0 0 0" rpy="0 0 0"/>
+      <parent link="${parent_link}"/>
+      <child link="${sensor_name}_link"/>
+      <axis xyz="0 0 1"/>
     </joint>
   </xacro:macro>
@@ -50,13 +52,16 @@
       <visual name="${sensor_name}_visual">
         <geometry>
-          <box><size>0.03 0.03 0.03</size></box>
+          <box size="0.03 0.03 0.03"/>
         </geometry>
       </visual>
       <inertial>
-        <mass>0.05</mass>
-        <inertia>
+        <mass value="0.05"/>
+        <inertia ixx="0.1" ixy="0.0" ixz="0.0"
+           iyy="0.1" iyz="0.0"
+           izz="0.1"/>
+        <!--<inertia>
           <ixx>1e-5</ixx><iyy>1e-5</iyy><izz>1e-5</izz>
           <ixy>0</ixy><ixz>0</ixz><iyz>0</iyz>
-        </inertia>
+        </inertia>-->
       </inertial>
       <sensor name="imu_sensor" type="imu">
@@ -69,11 +74,9 @@
     </link>
     <joint name="${sensor_name}_joint" type="fixed">
-      <parent>${parent_link}</parent>
-      <child>${sensor_name}_link</child>
-      <pose>0 0 0 0 0 0</pose>
-      <axis>
-        <xyz>0 0 1</xyz>
-      </axis>
+      <origin xyz="0 0 0" rpy="0 0 0"/>
+      <parent link="${parent_link}"/>
+      <child link="${sensor_name}_link"/>
+      <axis xyz="0 0 1"/>
     </joint>
   </xacro:macro>
-</sdf>
+</robot>

File: trackbot_gazebo/models/trackbot_vehicle/bogie.xacro (robot description, xacro)
@@ -1,4 +1,4 @@
 <?xml version="1.0"?>
-<sdf version="1.6" xmlns:xacro="http://ros.org/wiki/xacro">
+<robot xmlns:xacro="http://ros.org/wiki/xacro">
     <!-- Macro for a wheel -->
     <xacro:macro name="bogie_wheel" params="
@@ -35,36 +35,28 @@
       <xacro:property name="susp_izz" value="${1.0/12.0 * susp_mass * (3 * susp_r * susp_r + susp_l * susp_l)}"/>
       <xacro:property name="susp_joint_xyz" value="${x} ${y} ${z+susp_length/2}"/>
-      <xacro:property name="wheel_joint_xyz" value="${x} ${y_wheel} ${z - susp_length/2 + wheel_r}"/>
+      <xacro:property name="wheel_joint_xyz" value="${0} ${y_wheel} ${-susp_length/2}"/>
       <!-- =========================== -->
       <!-- Suspension Link             -->
       <!-- =========================== -->
       <link name="${name}_suspension_link">
-        <pose>0 0 0 0 0 0</pose>
         <inertial>
-          <mass>${susp_mass}</mass>
-          <inertia>
-            <ixx>${susp_ixx}</ixx><ixy>0</ixy><ixz>0</ixz>
-            <iyy>${susp_iyy}</iyy><iyz>0</iyz>
-            <izz>${susp_izz}</izz>
-          </inertia>
+          <mass value="${susp_mass}"/>
+          <inertia ixx="${susp_ixx}" ixy="0.0" ixz="0.0"
+            iyy="${susp_iyy}" iyz="0.0"
+            izz="${susp_izz}"/>
         </inertial>
         <collision name="${name}_suspension_collision">
-          <pose>${susp_joint_xyz} 0 0 0</pose> <!-- Rotate cylinder to face +Y -->
+          <origin xyz="0 0 0" rpy="0 0 0"/> <!-- Rotate cylinder to face +Y -->
           <geometry>
-            <cylinder>
-              <radius>${susp_r}</radius>
-              <length>${susp_l}</length>
-            </cylinder>
+            <cylinder radius="${susp_r}" length="${susp_l}"/>
           </geometry>
         </collision>
         <visual name="${name}_suspension_visual">
-          <pose>${susp_joint_xyz} 0 0 0</pose>
+          <origin xyz="0 0 0" rpy="0 0 0"/>
           <geometry>
-            <cylinder>
-              <radius>${susp_r}</radius>
-              <length>${susp_l}</length>
-            </cylinder>
+            <cylinder radius="${susp_r}" length="${susp_l}"/>
           </geometry>
-          <material>
+          <material name="suspension_color">
+            <color rgba="0.5 0.5 0.5 1.0"/>
             <ambient>0 0 1 1</ambient>
             <diffuse>0 0 1 1</diffuse>
@@ -76,31 +68,38 @@
       <!-- =========================== -->
       <joint name="${name}_suspension_joint" type="prismatic">
-        <pose>${susp_joint_xyz} 0 0 0</pose>
-        <parent>${parent_link}</parent>
-        <child>${name}_suspension_link</child>
+        <origin xyz="${x} ${y} ${z}" rpy="0 0 0"/>
+        <parent link="${parent_link}"/>
+        <child link="${name}_suspension_link"/>
+        <axis xyz="0 0 -1"/> <!-- moves along -Z -->
+        <limit lower="-0.1" upper="0.1" effort="500" velocity="10.0"/>
+        <!--<dynamics damping="${damping_coeff}" spring_stiffness="${spring_coeff}"/>--> <!--no springs-->
+      </joint>
+      <!-- Gazebo: dynamics only (NO <axis> wrapper to avoid duplication) -->
+      <xacro:if value="$(arg use_gazebo)">
+        <gazebo reference="${name}_suspension_joint">
         <axis>
-          <xyz>0 0 -1</xyz>
-          <limit>
-            <effort>100</effort>
-            <velocity>10.0</velocity>
-            <lower>-0.07</lower>
-            <upper>0.07</upper>
-            <stiffness>${spring_coeff}</stiffness>
-            <dissipation>0</dissipation>
-          </limit>
+          <dynamics>
+            <damping>${damping_coeff}</damping>
+            <spring_reference>0</spring_reference>
+            <spring_stiffness>${spring_coeff}</spring_stiffness>
+          </dynamics>
         </axis>
-        <physics>
-          <ode>
+          <!--<axis>
+            <xyz>0 0 -1</xyz>
             <limit>
-              <cfm>0.0</cfm>
-              <erp>0.2</erp>
+              <lower>-0.07</lower>
+              <upper>0.07</upper>
+              <effort>100</effort>
+              <velocity>10.0</velocity>
             </limit>
-          </ode>
-        </physics>
-        <dynamics>
-          <damping>${damping_coeff}</damping>
-          <spring_stiffness>${spring_coeff}</spring_stiffness>
-        </dynamics>
-      </joint>
+            <dynamics>
+              <damping>${damping_coeff}</damping>
+              <spring_reference>0</spring_reference>
+              <spring_stiffness>${spring_coeff}</spring_stiffness>
+            </dynamics>
+          </axis>
+          -->
+        </gazebo>
+      </xacro:if>
       <!-- =========================== -->
       <!-- wheel Link                  -->
@@ -108,29 +107,22 @@
       <link name="${name}_wheel_link">
         <inertial>
-          <mass>${wheel_mass}</mass>
-          <inertia>
-            <ixx>${wheel_ixx}</ixx><ixy>0</ixy><ixz>0</ixz>
-            <iyy>${wheel_iyy}</iyy><iyz>0</iyz>
-            <izz>${wheel_izz}</izz>
-          </inertia>
+          <mass value="${wheel_mass}"/>
+          <inertia ixx="${wheel_ixx}" ixy="0.0" ixz="0.0"
+            iyy="${wheel_iyy}" iyz="0.0"
+            izz="${wheel_izz}"/>
         </inertial>
         <collision name="${name}_wheel_collision">
-          <pose>${wheel_joint_xyz} 1.5708 0 0</pose>
+          <origin xyz="0 0 0" rpy="1.5708 0 0"/><!-- only rotate the cylinder -->
           <geometry>
-            <cylinder>
-              <radius>${wheel_r}</radius>
-              <length>${wheel_l}</length>
-            </cylinder>
+            <cylinder radius="${wheel_r}" length="${wheel_l}"/>
           </geometry>
         </collision>
         <visual name="${name}_wheel_visual">
-          <pose>${wheel_joint_xyz} 1.5708 0 0</pose>
+          <origin xyz="0 0 0" rpy="1.5708 0 0"/>
           <geometry>
-            <cylinder>
-              <radius>${wheel_r}</radius>
-              <length>${wheel_l}</length>
-            </cylinder>
+            <cylinder radius="${wheel_r}" length="${wheel_l}"/>
           </geometry>
-          <material>
+          <material name="bogie_wheel_color">
+            <color rgba="0.5 0.5 0.5 1.0"/>
             <ambient>0 0 1 1</ambient>
             <diffuse>0 0 1 1</diffuse>
@@ -141,14 +133,10 @@
       <!-- wheel Revolute Joint        -->
       <!-- =========================== -->
-      <joint name="${name}_wheel_joint" type="revolute">
-        <pose>${wheel_joint_xyz} 1.5708 0 0</pose>
-        <parent>${name}_suspension_link</parent>
-        <child>${name}_wheel_link</child>
-        <axis>
-          <xyz>0 1 0</xyz>
-        </axis>
-        <limit effort="10" velocity="10" lower="-3.14" upper="3.14"/>
-        <dynamics damping="0.1" friction="0.1"/>
+      <joint name="${name}_wheel_joint" type="continuous">
+        <origin xyz="${wheel_joint_xyz}" rpy="0 0 0"/> <!-- the *only* translation -->
+        <parent link="${name}_suspension_link"/>
+        <child link="${name}_wheel_link"/>
+        <axis xyz="0 1 0"/>
       </joint>
     </xacro:macro>
-</sdf>
+</robot>

File: trackbot_gazebo/models/trackbot_vehicle/model.urdf.xacro (robot description, xacro)
@@ -1,7 +1,8 @@
 <?xml version="1.0"?>
-<sdf version="1.6" xmlns:xacro="http://ros.org/wiki/xacro">
+<robot name="trackbot_vehicle" xmlns:xacro="http://ros.org/wiki/xacro">
   <xacro:include filename="wheel.xacro" />
   <xacro:include filename="bogie.xacro" />
   <xacro:include filename="../trackbot_sensors/sensors.xacro" />
+  <xacro:arg name="use_gazebo" default="false"/>
   <xacro:property name="body_length" value="1.8"/>
   <xacro:property name="body_width" value="0.96"/>
@@ -14,5 +15,4 @@
   <xacro:property name="drive_wheel_offset_y" value="${body_width/2+drive_wheel_w/2}"/>
   <xacro:property name="drive_wheel_offset_z" value="0.15"/>
-  <xacro:property name="bogie_wheel_offset_y" value="${body_width/2}"/>
   <xacro:property name="bogie_offset_z" value="0.0"/>
   <xacro:property name="bogie_wheel_d" value="0.2"/>
@@ -20,4 +20,5 @@
   <xacro:property name="bogie_wheel_mass" value="5.0"/>
   <xacro:property name="bogie_susp_d" value="0.1"/>
+  <xacro:property name="bogie_wheel_offset_y" value="${body_width/2+bogie_susp_d/2}"/>
   <xacro:property name="bogie_susp_l" value="0.2"/>
   <xacro:property name="bogie_susp_mass" value="1.0"/>
@@ -28,25 +29,20 @@
   <xacro:property name="lidar_front_xyz" value="0.9 0 0.4"/>
   <xacro:property name="lidar_front_rpy" value="0 0 0"/>
-  <model name="trackbot_vehicle">
-    <static>false</static>
+    <!-- Dummy root link with no inertia -->
+    <link name="root"/>
     <!-- ****************** ROBOT BASE FOOTPRINT ***************************  -->
-    <pose>0.0 0.0 0.0 0.0 0.0 0.0</pose>
     <link name="base_footprint"/>
     <!-- Base Link -->
     <link name="base_link">
-      <pose>0 0 ${body_height/2} 0 0 0</pose>
       <inertial>
-        <mass>${body_mass}</mass>
-        <inertia>
-          <ixx>1.0</ixx><ixy>0.0</ixy><ixz>0.0</ixz>
-          <iyy>1.0</iyy><iyz>0.0</iyz>
-          <izz>1.0</izz>
-        </inertia>
+        <mass value="${body_mass}"/>
+        <inertia ixx="${body_mass/12*(body_width*body_width+body_height*body_height)}" ixy="0.0" ixz="0.0"
+                iyy="${body_mass/12*(body_length*body_length+body_height*body_height)}" iyz="0.0"
+                izz="${body_mass/12*(body_length*body_length+body_width*body_width)}"/>
       </inertial>
       <collision name="base_collision">
+        <origin xyz="0 0 0.15" rpy="0 0 0"/>
         <geometry>
-          <box>
-            <size>${body_length} ${body_width} ${body_height}</size>
-          </box>
+          <box size="${body_length} ${body_width} ${body_height}"/>
         </geometry>
       </collision>
@@ -54,32 +50,40 @@
         <origin xyz="0 0 0.15" rpy="0 0 0"/>
         <geometry>
-          <mesh>
-          <uri>model://trackbot_vehicle/meshes/robot_base.stl</uri>
-          <scale>0.001 0.001 0.001</scale>
-          </mesh>
+          <box size="${body_length} ${body_width} ${body_height}"/>
+          <!--<mesh filename="package://trackbot_gazebo/models/trackbot_vehicle/meshes/robot_base.stl" scale="0.001 0.001 0.001"/>
+          <xacro:if value="$(arg use_gazebo)">
+            <mesh>
+              <uri>model://trackbot_vehicle/meshes/robot_base.stl</uri>
+            </mesh>
+          </xacro:if>
+          <xacro:unless value="$(arg use_gazebo)">
+            <mesh filename="package://trackbot_gazebo/models/trackbot_vehicle/meshes/robot_base.stl"/>
+          </xacro:unless>-->
         </geometry>
-        <material>
-          <ambient>1.0 0.0 0.0 1.0</ambient>
-          <diffuse>1.0 0.0 0.0 1.0</diffuse>
-          <specular>0.2 0.2 0.2 1.0</specular>
-          <emissive>0.0 0.0 0.0 1.0</emissive>
-      </material>
+        <material name="body_color">
+          <color rgba="0.5 0.5 0.5 1.0"/>
+        </material>
       </visual>
     </link>
     <!-- ************************ JOINTS ***********************************  -->
-    <!-- Pose of the joint is the same as the child link frame -->
-    <!-- Axis is the axis of rotation relative to the child link frame -->
+    <!-- Your original root becomes a child -->
+    <joint name="root_to_base" type="fixed">
+      <parent link="root"/>
+      <child link="base_footprint"/>
+    </joint>
     <joint name="base_joint" type="fixed">
-      <parent>base_footprint</parent>
-      <child>base_link</child>
-      <pose>0 0 0 0 0 0</pose>
+      <origin xyz="0 0 0" rpy="0 0 0"/>
+      <parent link="base_footprint"/>
+      <child link="base_link"/>
     </joint>
-    <plugin name="gz::sim::systems::Sensors"
-        filename="gz-sim-sensors-system">
-    </plugin>
-    <plugin
-      filename="gz-sim-imu-system"
-      name="gz::sim::systems::Imu">
-    </plugin>
+    <gazebo>
+      <plugin name="gz::sim::systems::Sensors"
+          filename="gz-sim-sensors-system">
+      </plugin>
+      <plugin
+        filename="gz-sim-imu-system"
+        name="gz::sim::systems::Imu">
+      </plugin>
+    </gazebo>
     <xacro:camera_sensor sensor_name="front_camera" parent_link="base_link" pose="${camera_front_xyz}" rpy="${camera_front_rpy}"/>
     <xacro:imu_sensor sensor_name="inertial_unit" parent_link="base_link"/>
@@ -96,6 +100,5 @@
     <xacro:bogie_wheel name="bogie_left_1" parent_link="base_link"
         x="0.5" y="${bogie_wheel_offset_y}" z="${bogie_offset_z}"
-        y_wheel="${bogie_wheel_offset_y + bogie_susp_d/2 + bogie_wheel_w/2}"
-        rpy="0 0 0"
+        y_wheel="${bogie_susp_d/2 + bogie_wheel_w/2}" rpy="0 0 0"
         wheel_diameter="${bogie_wheel_d}" wheel_length="${bogie_wheel_w}" wheel_mass="${bogie_wheel_mass}"
         susp_diameter="${bogie_susp_d}" susp_length="${bogie_susp_l}" susp_mass="${bogie_susp_mass}"
@@ -103,6 +106,5 @@
     <xacro:bogie_wheel name="bogie_left_2" parent_link="base_link"
         x="0.0" y="${bogie_wheel_offset_y}" z="${bogie_offset_z}"
-        y_wheel="${bogie_wheel_offset_y + bogie_susp_d/2 + bogie_wheel_w/2}"
-        rpy="0 0 0"
+        y_wheel="${bogie_susp_d/2 + bogie_wheel_w/2}" rpy="0 0 0"
         wheel_diameter="${bogie_wheel_d}" wheel_length="${bogie_wheel_w}" wheel_mass="${bogie_wheel_mass}"
         susp_diameter="${bogie_susp_d}" susp_length="${bogie_susp_l}" susp_mass="${bogie_susp_mass}"
@@ -110,13 +112,11 @@
     <xacro:bogie_wheel name="bogie_left_3" parent_link="base_link"
         x="-0.5" y="${bogie_wheel_offset_y}" z="${bogie_offset_z}"
-        y_wheel="${bogie_wheel_offset_y + bogie_susp_d/2 + bogie_wheel_w/2}"
-        rpy="0 0 0"
-        wheel_diameter="${bogie_wheel_d}" wheel_length="${bogie_wheel_w}" wheel_mass="${bogie_wheel_mass}"
+        y_wheel="${bogie_susp_d/2 + bogie_wheel_w/2}" rpy="0 0 0"
+        wheel_diameter="${bogie_wheel_d}"  wheel_length="${bogie_wheel_w}" wheel_mass="${bogie_wheel_mass}"
         susp_diameter="${bogie_susp_d}" susp_length="${bogie_susp_l}" susp_mass="${bogie_susp_mass}"
         spring_coeff="${bogie_spring_coeff}" damping_coeff="${bogie_damping_coeff}"/>
     <xacro:bogie_wheel name="bogie_right_1" parent_link="base_link"
         x="0.5" y="${-bogie_wheel_offset_y}" z="${bogie_offset_z}"
-        y_wheel="${-bogie_wheel_offset_y - bogie_susp_d/2 - bogie_wheel_w/2}"
-        rpy="0 0 0"
+        y_wheel="${-bogie_susp_d/2 - bogie_wheel_w/2}" rpy="0 0 0"
         wheel_diameter="${bogie_wheel_d}" wheel_length="${bogie_wheel_w}" wheel_mass="${bogie_wheel_mass}"
         susp_diameter="${bogie_susp_d}" susp_length="${bogie_susp_l}" susp_mass="${bogie_susp_mass}"
@@ -124,6 +124,5 @@
     <xacro:bogie_wheel name="bogie_right_2" parent_link="base_link"
         x="0.0" y="${-bogie_wheel_offset_y}" z="${bogie_offset_z}"
-        y_wheel="${-bogie_wheel_offset_y - bogie_susp_d/2 - bogie_wheel_w/2}"
-        rpy="0 0 0"
+        y_wheel="${-bogie_susp_d/2 - bogie_wheel_w/2}" rpy="0 0 0"
         wheel_diameter="${bogie_wheel_d}" wheel_length="${bogie_wheel_w}" wheel_mass="${bogie_wheel_mass}"
         susp_diameter="${bogie_susp_d}" susp_length="${bogie_susp_l}" susp_mass="${bogie_susp_mass}"
@@ -131,6 +130,5 @@
     <xacro:bogie_wheel name="bogie_right_3" parent_link="base_link"
         x="-0.5" y="${-bogie_wheel_offset_y}" z="${bogie_offset_z}"
-        y_wheel="${-bogie_wheel_offset_y - bogie_susp_d/2 - bogie_wheel_w/2}"
-        rpy="0 0 0"
+        y_wheel="${-bogie_susp_d/2 - bogie_wheel_w/2}" rpy="0 0 0"
         wheel_diameter="${bogie_wheel_d}" wheel_length="${bogie_wheel_w}" wheel_mass="${bogie_wheel_mass}"
         susp_diameter="${bogie_susp_d}" susp_length="${bogie_susp_l}" susp_mass="${bogie_susp_mass}"
@@ -138,9 +136,15 @@
     <!-- Plugin to use ROS2 DiffDrive -->
     <plugin filename="gz-sim-diff-drive-system" name="gz::sim::systems::DiffDrive">
-      <!-- wheels -->
+      <!-- wheels
       <left_joint>drivewhl_left_f_joint</left_joint>
       <left_joint>drivewhl_left_r_joint</left_joint>
       <right_joint>drivewhl_right_f_joint</right_joint>
-      <right_joint>drivewhl_right_r_joint</right_joint>
+      <right_joint>drivewhl_right_r_joint</right_joint>-->
+      <left_joint>bogie_left_1_wheel_joint</left_joint>
+      <left_joint>bogie_left_2_wheel_joint</left_joint>
+      <left_joint>bogie_left_3_wheel_joint</left_joint>
+      <right_joint>bogie_right_1_wheel_joint</right_joint>
+      <right_joint>bogie_right_2_wheel_joint</right_joint>
+      <right_joint>bogie_right_3_wheel_joint</right_joint>
       <!-- kinematics -->
       <wheel_separation>${2 * drive_wheel_offset_y}</wheel_separation>
@@ -183,4 +187,3 @@
       <joint_name>bogie_right_3_wheel_joint</joint_name>
     </plugin>
-  </model>
-</sdf>
+</robot>

File: trackbot_gazebo/models/trackbot_vehicle/wheel.xacro (robot description, xacro)
@@ -1,4 +1,4 @@
 <?xml version="1.0"?>
-<sdf version="1.6" xmlns:xacro="http://ros.org/wiki/xacro">
+<robot xmlns:xacro="http://ros.org/wiki/xacro">
     <!-- Macro for a wheel -->
     <xacro:macro name="drive_wheel" params="
@@ -11,42 +11,32 @@
         z:='0'
         ">
-      <xacro:property name="wheel_radius" value="${wheel_diameter/2}"/>
-      <xacro:property name="wheel_width" value="${wheel_length}"/>
-      <link name="${name}_link">
-        <pose>0 0 0 0 0 0</pose>
-        <inertial>
-          <mass>${wheel_mass}</mass>
-          <inertia>
-            <ixx>0.01</ixx><ixy>0</ixy><ixz>0</ixz>
-            <iyy>0.01</iyy><iyz>0</iyz><izz>0.01</izz>
-          </inertia>
-        </inertial>
-        <collision name="${name}_collision">
-          <pose>${x} ${y} ${z} 1.5708 0 0</pose> <!-- Rotate cylinder to face +Y -->
-          <geometry>
-            <cylinder>
-              <radius>${wheel_radius}</radius>
-              <length>${wheel_width}</length>
-            </cylinder>
-          </geometry>
-        </collision>
-        <visual name="${name}_visual">
-          <pose>${x} ${y} ${z} 1.5708 0 0</pose> <!-- Rotate cylinder to face +Y -->
-          <geometry>
-            <cylinder>
-              <radius>${wheel_radius}</radius>
-              <length>${wheel_width}</length>
-            </cylinder>
-          </geometry>
-        </visual>
-      </link>
-      <joint name="${name}_joint" type="revolute">
-        <pose>${x} ${y} ${z} 0 0 0</pose>
-        <parent>base_link</parent>
-        <child>${name}_link</child>
-        <axis>
-          <xyz>0 1 0</xyz>
-        </axis>
-      </joint>
-    </xacro:macro>
-</sdf>
+    <xacro:property name="wheel_radius" value="${wheel_diameter/2}"/>
+    <xacro:property name="wheel_width" value="${wheel_length}"/>
+    <link name="${name}_link">
+      <inertial>
+        <mass value="${wheel_mass}"/>
+        <inertia ixx="0.1" ixy="0.0" ixz="0.0"
+                iyy="0.1" iyz="0.0"
+                izz="0.1"/>
+      </inertial>
+      <collision name="${name}_collision">
+        <origin xyz="${x} ${y} ${z}" rpy="1.5708 0 0"/> <!-- Rotate cylinder to face +Y -->
+        <geometry>
+          <cylinder radius="${wheel_radius}" length="${wheel_width}"/>
+        </geometry>
+      </collision>
+      <visual name="${name}_visual">
+        <origin xy="${x} ${y} ${z}" rpy="1.5708 0 0"/> <!-- Rotate cylinder to face +Y -->
+        <geometry>
+          <cylinder radius="${wheel_radius}" length="${wheel_width}"/>
+        </geometry>
+      </visual>
+    </link>
+    <joint name="${name}_joint" type="continuous">
+      <origin xyz="${x} ${y} ${z}" rpy="0 0 0"/>
+      <parent link="base_link"/>
+      <child link="${name}_link"/>
+      <axis xyz="0 1 0"/>
+    </joint>
+  </xacro:macro>
+</robot>
