Commit message: Modified launch files, sensors etc

File: trackbot_gazebo/models/trackbot_sensors/sensors.xacro (robot description, xacro)
@@ -1,82 +1,65 @@
 <?xml version="1.0"?>
 <robot xmlns:xacro="http://ros.org/wiki/xacro">
-  <xacro:macro name="camera_sensor" params="sensor_name parent_link pose rpy">
+  <!-- Camera -->
+  <xacro:macro name="camera_sensor" params="sensor_name parent_link xyz:='0 0 0' rpy:='0 0 0'">
     <link name="${sensor_name}_link">
-      <pose>${pose} ${rpy}</pose>
       <visual name="${sensor_name}_visual">
-        <geometry>
-          <box size="0.05 0.05 0.05"/>
-        </geometry>
-        <material name="camera_color">
-          <color rgba="0.5 0.5 0.5 1.0"/>
-          <ambient>1.0 1.0 0.0 1.0</ambient>
-          <diffuse>1.0 1.0 0.0 1.0</diffuse>
-          <specular>0.2 0.2 0.2 1.0</specular>
-          <emissive>0.0 0.0 0.0 1.0</emissive>
-        </material>
+        <geometry><box size="0.05 0.05 0.05"/></geometry>
       </visual>
       <inertial>
         <mass value="0.1"/>
-        <inertia ixx="0.1" ixy="0.0" ixz="0.0"
-           iyy="0.1" iyz="0.0"
-           izz="0.1"/>
-        <!--<inertia>
-          <ixx>1e-5</ixx><iyy>1e-5</iyy><izz>1e-5</izz>
-          <ixy>0</ixy><ixz>0</ixz><iyz>0</iyz>
-        </inertia>-->
+        <inertia ixx="1e-5" ixy="0" ixz="0" iyy="1e-5" iyz="0" izz="1e-5"/>
       </inertial>
+    </link>
+    <joint name="${sensor_name}_joint" type="fixed">
+      <parent link="${parent_link}"/>
+      <child  link="${sensor_name}_link"/>
+      <origin xyz="${xyz}" rpy="${rpy}"/>
+    </joint>
+    <!-- SDF sensor lives under a gazebo block, referenced to the link -->
+    <gazebo reference="${sensor_name}_link">
       <sensor name="${sensor_name}" type="camera">
         <always_on>true</always_on>
         <update_rate>30</update_rate>
         <visualize>true</visualize>
-        <topic>camera/image_raw</topic>
-        <gz_frame_id>camera_rgb_frame</gz_frame_id>
+        <!-- Set an explicit topic; Gazebo will still scope it under /model/<name>/... -->
+        <topic>/camera/image_raw</topic>
+        <gz_frame_id>${sensor_name}_link</gz_frame_id>
         <camera>
-          <camera_info_topic>camera/camera_info</camera_info_topic>
+          <camera_info_topic>/camera/camera_info</camera_info_topic>
           <horizontal_fov>1.047</horizontal_fov>
-          <image><width>640</width><height>480</height><format>R8G8B8</format></image>
+          <image>
+            <width>640</width><height>480</height><format>R8G8B8</format>
+          </image>
           <clip><near>0.1</near><far>100</far></clip>
         </camera>
       </sensor>
-    </link>
-    <joint name="${sensor_name}_joint" type="fixed">
-      <origin xyz="0 0 0" rpy="0 0 0"/>
-      <parent link="${parent_link}"/>
-      <child link="${sensor_name}_link"/>
-      <axis xyz="0 0 1"/>
-    </joint>
+    </gazebo>
   </xacro:macro>
-  <xacro:macro name="imu_sensor" params="sensor_name parent_link pose_xyz:='0 0 0.2' pose_rpy:='0 0 0'">
+  <!-- IMU -->
+  <xacro:macro name="imu_sensor" params="sensor_name parent_link xyz:='0 0 0.2' rpy:='0 0 0'">
     <link name="${sensor_name}_link">
-      <pose>${pose_xyz} ${pose_rpy}</pose>
       <visual name="${sensor_name}_visual">
-        <geometry>
-          <box size="0.03 0.03 0.03"/>
-        </geometry>
+        <geometry><box size="0.03 0.03 0.03"/></geometry>
       </visual>
       <inertial>
         <mass value="0.05"/>
-        <inertia ixx="0.1" ixy="0.0" ixz="0.0"
-           iyy="0.1" iyz="0.0"
-           izz="0.1"/>
-        <!--<inertia>
-          <ixx>1e-5</ixx><iyy>1e-5</iyy><izz>1e-5</izz>
-          <ixy>0</ixy><ixz>0</ixz><iyz>0</iyz>
-        </inertia>-->
+        <inertia ixx="1e-5" ixy="0" ixz="0" iyy="1e-5" iyz="0" izz="1e-5"/>
       </inertial>
-      <sensor name="imu_sensor" type="imu">
+    </link>
+    <joint name="${sensor_name}_joint" type="fixed">
+      <parent link="${parent_link}"/>
+      <child  link="${sensor_name}_link"/>
+      <origin xyz="${xyz}" rpy="${rpy}"/>
+    </joint>
+    <gazebo reference="${sensor_name}_link">
+      <sensor name="${sensor_name}" type="imu">
+        <always_on>true</always_on>
+        <update_rate>100</update_rate>
+        <visualize>true</visualize>
         <topic>/imu/data</topic>
-        <update_rate>100.0</update_rate>
-        <always_on>1</always_on>
-        <visualize>1</visualize>
         <gz_frame_id>${sensor_name}_link</gz_frame_id>
       </sensor>
-    </link>
-    <joint name="${sensor_name}_joint" type="fixed">
-      <origin xyz="0 0 0" rpy="0 0 0"/>
-      <parent link="${parent_link}"/>
-      <child link="${sensor_name}_link"/>
-      <axis xyz="0 0 1"/>
-    </joint>
+    </gazebo>
   </xacro:macro>
 </robot>

File: trackbot_gazebo/models/trackbot_vehicle/model.urdf.xacro (robot description, xacro)
@@ -50,14 +50,7 @@
         <origin xyz="0 0 0.15" rpy="0 0 0"/>
         <geometry>
-          <box size="${body_length} ${body_width} ${body_height}"/>
-          <!--<mesh filename="package://trackbot_gazebo/models/trackbot_vehicle/meshes/robot_base.stl" scale="0.001 0.001 0.001"/>
-          <xacro:if value="$(arg use_gazebo)">
-            <mesh>
-              <uri>model://trackbot_vehicle/meshes/robot_base.stl</uri>
-            </mesh>
-          </xacro:if>
-          <xacro:unless value="$(arg use_gazebo)">
-            <mesh filename="package://trackbot_gazebo/models/trackbot_vehicle/meshes/robot_base.stl"/>
-          </xacro:unless>-->
+          <!-- Use model:// with the *model name* that has model.config -->
+          <mesh filename="package://trackbot_vehicle/meshes/robot_base.stl"
+                scale="0.001 0.001 0.001"/>
         </geometry>
         <material name="body_color">
@@ -86,5 +79,5 @@
       </plugin>
     </gazebo>
-    <xacro:camera_sensor sensor_name="front_camera" parent_link="base_link" pose="${camera_front_xyz}" rpy="${camera_front_rpy}"/>
+    <xacro:camera_sensor sensor_name="front_camera" parent_link="base_link" xyz="${camera_front_xyz}" rpy="${camera_front_rpy}"/>
     <xacro:imu_sensor sensor_name="inertial_unit" parent_link="base_link"/>
     <!-- Instantiate four drive wheels -->
@@ -135,55 +128,59 @@
         spring_coeff="${bogie_spring_coeff}" damping_coeff="${bogie_damping_coeff}"/>
     <!-- Plugin to use ROS2 DiffDrive -->
-    <plugin filename="gz-sim-diff-drive-system" name="gz::sim::systems::DiffDrive">
-      <!-- wheels
-      <left_joint>drivewhl_left_f_joint</left_joint>
-      <left_joint>drivewhl_left_r_joint</left_joint>
-      <right_joint>drivewhl_right_f_joint</right_joint>
-      <right_joint>drivewhl_right_r_joint</right_joint>-->
-      <left_joint>bogie_left_1_wheel_joint</left_joint>
-      <left_joint>bogie_left_2_wheel_joint</left_joint>
-      <left_joint>bogie_left_3_wheel_joint</left_joint>
-      <right_joint>bogie_right_1_wheel_joint</right_joint>
-      <right_joint>bogie_right_2_wheel_joint</right_joint>
-      <right_joint>bogie_right_3_wheel_joint</right_joint>
-      <!-- kinematics -->
-      <wheel_separation>${2 * drive_wheel_offset_y}</wheel_separation>
-      <wheel_radius>${drive_wheel_d}/2</wheel_radius>
-      <!-- limits -->
-      <max_linear_acceleration>1.0</max_linear_acceleration>
-      <topic>cmd_vel</topic>
-      <odom_topic>odom</odom_topic>
-      <frame_id>odom</frame_id>
-      <tf_topic>/tf</tf_topic>
-      <odom_publisher_frequency>30</odom_publisher_frequency>
-      <child_frame_id>base_footprint</child_frame_id>
-      <ros>
-          <namespace>/</namespace>        <!-- put ROS topics at root -->
-          <remapping>cmd_vel:=cmd_vel</remapping>
-          <remapping>odom:=odom</remapping>
-      </ros>
-    </plugin>
+    <gazebo>
+      <plugin filename="gz-sim-diff-drive-system" name="gz::sim::systems::DiffDrive">
+        <!-- wheels
+        <left_joint>drivewhl_left_f_joint</left_joint>
+        <left_joint>drivewhl_left_r_joint</left_joint>
+        <right_joint>drivewhl_right_f_joint</right_joint>
+        <right_joint>drivewhl_right_r_joint</right_joint>-->
+        <left_joint>bogie_left_1_wheel_joint</left_joint>
+        <left_joint>bogie_left_2_wheel_joint</left_joint>
+        <left_joint>bogie_left_3_wheel_joint</left_joint>
+        <right_joint>bogie_right_1_wheel_joint</right_joint>
+        <right_joint>bogie_right_2_wheel_joint</right_joint>
+        <right_joint>bogie_right_3_wheel_joint</right_joint>
+        <!-- kinematics -->
+        <wheel_separation>${2 * drive_wheel_offset_y}</wheel_separation>
+        <wheel_radius>${drive_wheel_d}/2</wheel_radius>
+        <!-- limits -->
+        <max_linear_acceleration>1.0</max_linear_acceleration>
+        <topic>cmd_vel</topic>
+        <odom_topic>odom</odom_topic>
+        <frame_id>odom</frame_id>
+        <tf_topic>/tf</tf_topic>
+        <odom_publisher_frequency>30</odom_publisher_frequency>
+        <child_frame_id>base_footprint</child_frame_id>
+        <ros>
+            <namespace>/</namespace>        <!-- put ROS topics at root -->
+            <remapping>cmd_vel:=cmd_vel</remapping>
+            <remapping>odom:=odom</remapping>
+        </ros>
+      </plugin>
+    </gazebo>
     <!-- Plugin to publish joint states and broadcast TF -->
-    <plugin filename="gz-sim-joint-state-publisher-system" name="gz::sim::systems::JointStatePublisher">
-      <topic>joint_states</topic>
-      <publish_frequency>50</publish_frequency>
-      <update_rate>30</update_rate>
-      <!--<joint_name_suffix>_joint</joint_name_suffix>-->
-      <joint_name>drivewhl_left_f_joint</joint_name>
-      <joint_name>drivewhl_right_f_joint</joint_name>
-      <joint_name>drivewhl_left_r_joint</joint_name>
-      <joint_name>drivewhl_right_r_joint</joint_name>
-      <joint_name>bogie_left_1_suspension_joint</joint_name>
-      <joint_name>bogie_left_2_suspension_joint</joint_name>
-      <joint_name>bogie_left_3_suspension_joint</joint_name>
-      <joint_name>bogie_right_1_suspension_joint</joint_name>
-      <joint_name>bogie_right_2_suspension_joint</joint_name>
-      <joint_name>bogie_right_3_suspension_joint</joint_name>
-      <joint_name>bogie_left_1_wheel_joint</joint_name>
-      <joint_name>bogie_left_2_wheel_joint</joint_name>
-      <joint_name>bogie_left_3_wheel_joint</joint_name>
-      <joint_name>bogie_right_1_wheel_joint</joint_name>
-      <joint_name>bogie_right_2_wheel_joint</joint_name>
-      <joint_name>bogie_right_3_wheel_joint</joint_name>
-    </plugin>
+    <gazebo>
+      <plugin filename="gz-sim-joint-state-publisher-system" name="gz::sim::systems::JointStatePublisher">
+        <topic>joint_states</topic>
+        <publish_frequency>50</publish_frequency>
+        <update_rate>30</update_rate>
+        <!--<joint_name_suffix>_joint</joint_name_suffix>-->
+        <joint_name>drivewhl_left_f_joint</joint_name>
+        <joint_name>drivewhl_right_f_joint</joint_name>
+        <joint_name>drivewhl_left_r_joint</joint_name>
+        <joint_name>drivewhl_right_r_joint</joint_name>
+        <joint_name>bogie_left_1_suspension_joint</joint_name>
+        <joint_name>bogie_left_2_suspension_joint</joint_name>
+        <joint_name>bogie_left_3_suspension_joint</joint_name>
+        <joint_name>bogie_right_1_suspension_joint</joint_name>
+        <joint_name>bogie_right_2_suspension_joint</joint_name>
+        <joint_name>bogie_right_3_suspension_joint</joint_name>
+        <joint_name>bogie_left_1_wheel_joint</joint_name>
+        <joint_name>bogie_left_2_wheel_joint</joint_name>
+        <joint_name>bogie_left_3_wheel_joint</joint_name>
+        <joint_name>bogie_right_1_wheel_joint</joint_name>
+        <joint_name>bogie_right_2_wheel_joint</joint_name>
+        <joint_name>bogie_right_3_wheel_joint</joint_name>
+      </plugin>
+    </gazebo>
 </robot>
